File: pcb/EAQM-250201.kicad_sch (KiCad schematic)
At the start: 44 parts, among them J1 TYPE-C-31-M-12, J2 SSD1306, J3 Conn_01x04_Socket, J4 Conn_01x05_Socket, Q1 AO3418, Q2 AO3418, SW1 TS-1187A-B-A-B, SW2 TS-1187A-B-A-B, U1 LM1117MP-3.3, U2 BMP280, U3 SHT30-DIS, U4 ESP32-C6-MINI-1/U

Commit message: :sparkles: Update schematic
Parts:
- R7: value 22 -> 10k
- SW1, SW2: symbol Switch:SW_MEC_5E -> Switch:SW_Push
Connections:
- net Earth: no longer C1.2, C2.2, C3.2, C4.1, C5.2, C6.2, C7.2, C8.1, C9.2, J1.A1 (GND), J1.A12 (GND), J1.B1 (GND), J1.B12 (GND), J2.4 (Pin_4), J3.3 (Pin_3), R2.2, R3.2, R5.2, R6.2, SW1.1, SW1.2, SW2.3 (K), SW2.4 (A), TP3.1, TP4.1, U1.1 (GND), U2.1 (GND), U2.5 (SDO), U2.7 (GND), U3.2 (ADDR), U3.7 (R), U3.8 (VSS), U3.9 (VSS), U4.1 (GND), U4.11 (GND), U4.14 (GND), U4.2 (GND), U4.36 (GND), U4.37 (GND), U4.38 (GND), U4.39 (GND), U4.40 (GND), U4.41 (GND), U4.42 (GND), U4.43 (GND), U4.44 (GND), U4.45 (GND), U4.46 (GND), U4.47 (GND), U4.48 (GND), U4.49 (GND), U4.50 (GND), U4.51 (GND), U4.52 (GND), U4.53 (GND)
- net at C8.2, R8.2, U4.8 (EN/CHIP_PU): now also SW1.2; no longer SW1.3 (K), SW1.4 (A)
- net at C9.1, R10.2, SW2.1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: no longer SW2.2
- new net GND: C1.2, C2.2, C3.2, C4.1, C5.2, C6.2, C7.2, C8.1, C9.2, J1.A1 (GND), J1.A12 (GND), J1.B1 (GND), J1.B12 (GND), J2.4 (Pin_4), J3.3 (Pin_3), R2.2, R3.2, R5.2, R6.2, SW1.1, SW2.2, TP3.1, TP4.1, U1.1 (GND), U2.1 (GND), U2.5 (SDO), U2.7 (GND), U3.2 (ADDR), U3.7 (R), U3.8 (VSS), U3.9 (VSS), U4.1 (GND), U4.11 (GND), U4.14 (GND), U4.2 (GND), U4.36 (GND), U4.37 (GND), U4.38 (GND), U4.39 (GND), U4.40 (GND), U4.41 (GND), U4.42 (GND), U4.43 (GND), U4.44 (GND), U4.45 (GND), U4.46 (GND), U4.47 (GND), U4.48 (GND), U4.49 (GND), U4.50 (GND), U4.51 (GND), U4.52 (GND), U4.53 (GND)
Changed lines of the file:
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@@
 	)
 	(junction
-		(at 41.91 161.29)
-		(diameter 0)
-		(color 0 0 0 0)
-	)
-	(junction
 		(at 104.14 74.93)
 		(diameter 0)
@@
 	)
 	(junction
-		(at 57.15 158.75)
-		(diameter 0)
-		(color 0 0 0 0)
-	)
-	(junction
 		(at 307.34 181.61)
 		(diameter 0)
@@
 	)
 	(junction
-		(at 162.56 186.69)
-		(diameter 0)
-		(color 0 0 0 0)
-	)
-	(junction
 		(at 88.9 77.47)
 		(diameter 0)
@@
 	)
 	(junction
-		(at 177.8 186.69)
-		(diameter 0)
-		(color 0 0 0 0)
-	)
-	(junction
 		(at 67.31 67.31)
 		(diameter 0)
@@
 	(wire
 		(pts
-			(xy 54.61 158.75) (xy 57.15 158.75)
-		)
-		(stroke
-			(width 0)
-			(type default)
-		)
-	)
-	(wire
-		(pts
 			(xy 104.14 52.07) (xy 63.5 52.07)
 		)
@@
 	(wire
 		(pts
-			(xy 41.91 158.75) (xy 41.91 161.29)
-		)
-		(stroke
-			(width 0)
-			(type default)
-		)
-	)
-	(wire
-		(pts
 			(xy 147.32 46.99) (xy 156.21 46.99)
 		)
@@
 	(wire
 		(pts
-			(xy 177.8 184.15) (xy 177.8 186.69)
-		)
-		(stroke
-			(width 0)
-			(type default)
-		)
-	)
-	(wire
-		(pts
 			(xy 156.21 59.69) (xy 158.75 59.69)
 		)
@@
 	(wire
 		(pts
-			(xy 175.26 184.15) (xy 177.8 184.15)
-		)
-		(stroke
-			(width 0)
-			(type default)
-		)
-	)
-	(wire
-		(pts
 			(xy 123.19 59.69) (xy 123.19 62.23)
 		)
@@
 	(wire
 		(pts
-			(xy 162.56 184.15) (xy 162.56 186.69)
-		)
-		(stroke
-			(width 0)
-			(type default)
-		)
-	)
-	(wire
-		(pts
 			(xy 66.04 184.15) (xy 76.2 184.15)
 		)
@@
 	(wire
 		(pts
-			(xy 57.15 161.29) (xy 57.15 158.75)
-		)
-		(stroke
-			(width 0)
-			(type default)
-		)
-	)
-	(wire
-		(pts
 			(xy 173.99 45.72) (xy 182.88 45.72)
 		)
@@
 	(wire
 		(pts
-			(xy 54.61 161.29) (xy 57.15 161.29)
+			(xy 54.61 158.75) (xy 72.39 158.75)
 		)
 		(stroke
@@
 	(wire
 		(pts
-			(xy 40.64 101.6) (xy 50.8 101.6)
-		)
-		(stroke
-			(width 0)
-			(type default)
-		)
-	)
-	(wire
-		(pts
 			(xy 41.91 158.75) (xy 44.45 158.75)
 		)
@@
 	(wire
 		(pts
-			(xy 162.56 186.69) (xy 165.1 186.69)
-		)
-		(stroke
-			(width 0)
-			(type default)
-		)
-	)
-	(wire
-		(pts
 			(xy 307.34 201.93) (xy 297.18 201.93)
 		)
@@
 	(wire
 		(pts
-			(xy 160.02 186.69) (xy 162.56 186.69)
+			(xy 160.02 186.69) (xy 165.1 186.69)
 		)
 		(stroke
@@
 	(wire
 		(pts
-			(xy 157.48 175.26) (xy 157.48 176.53)
+			(xy 41.91 158.75) (xy 41.91 163.83)
 		)
 		(stroke
@@
 	(wire
 		(pts
-			(xy 55.88 179.07) (xy 55.88 180.34)
+			(xy 157.48 175.26) (xy 157.48 176.53)
 		)
 		(stroke
@@
 	(wire
 		(pts
-			(xy 345.44 77.47) (xy 345.44 78.74)
+			(xy 55.88 179.07) (xy 55.88 180.34)
 		)
 		(stroke
@@
 	(wire
 		(pts
-			(xy 40.64 104.14) (xy 40.64 101.6)
+			(xy 345.44 77.47) (xy 345.44 78.74)
 		)
 		(stroke
@@
 	(wire
 		(pts
-			(xy 165.1 184.15) (xy 162.56 184.15)
+			(xy 40.64 104.14) (xy 40.64 101.6)
 		)
 		(stroke
@@
 	(wire
 		(pts
-			(xy 57.15 158.75) (xy 72.39 158.75)
-		)
-		(stroke
-			(width 0)
-			(type default)
-		)
-	)
-	(wire
-		(pts
-			(xy 41.91 161.29) (xy 44.45 161.29)
-		)
-		(stroke
-			(width 0)
-			(type default)
-		)
-	)
-	(wire
-		(pts
 			(xy 283.21 181.61) (xy 283.21 184.15)
 		)
@@
 	(wire
 		(pts
-			(xy 41.91 161.29) (xy 41.91 163.83)
-		)
-		(stroke
-			(width 0)
-			(type default)
-		)
-	)
-	(wire
-		(pts
 			(xy 298.45 189.23) (xy 298.45 191.77)
 		)
@@
 	)
 	(rectangle
-		(start 167.64 173.355)
-		(end 172.72 175.895)
+		(start 167.767 174.752)
+		(end 172.847 177.292)
 		(stroke
 			(width 0)
@@
 	(text "BOOT"
 		(exclude_from_sim no)
-		(at 170.18 175.006 0)
+		(at 170.307 176.403 0)
 		(effects
 			(font
@@
 	)
 	(symbol
-		(lib_id "Switch:SW_MEC_5E")
+		(lib_id "Switch:SW_Push")
 		(at 170.18 186.69 0)
 		(unit 1)
@@
 		(dnp no)
 		(property "Reference" "SW2"
-			(at 169.418 179.578 0)
+			(at 167.386 180.848 0)
 			(effects
 				(font
@@
 		)
 		(property "Value" "TS-1187A-B-A-B"
-			(at 182.118 179.578 0)
+			(at 180.086 180.848 0)
 			(effects
 				(font
@@
 		)
 		(property "Footprint" "Button_Switch_SMD:SW_Push_1P1T_XKB_TS-1187A"
-			(at 170.18 179.07 0)
+			(at 170.18 181.61 0)
 			(effects
 				(font
@@
 			)
 		)
-		(property "Datasheet" "http://www.apem.com/int/index.php?controller=attachment&id_attachment=1371"
-			(at 170.18 179.07 0)
+		(property "Datasheet" "~"
+			(at 170.18 181.61 0)
 			(effects
 				(font
@@
 			)
 		)
-		(property "Description" "MEC 5E single pole normally-open tactile switch"
+		(property "Description" "Push button switch, generic, two pins"
 			(at 170.18 186.69 0)
 			(effects
@@
 		(pin "1"
 		)
-		(pin "4"
-		)
-		(pin "3"
-		)
 		(pin "2"
 		)
@@
 			)
 		)
-		(property "Value" "22"
+		(property "Value" "10k"
 			(at 242.316 69.088 90)
 			(effects
@@
 	)
 	(symbol
-		(lib_id "Switch:SW_MEC_5E")
-		(at 49.53 161.29 0)
+		(lib_id "Switch:SW_Push")
+		(at 49.53 158.75 0)
 		(unit 1)
 		(exclude_from_sim no)
@@
 		(dnp no)
 		(property "Reference" "SW1"
-			(at 39.878 154.178 0)
+			(at 39.624 153.67 0)
 			(effects
 				(font
@@
 		)
 		(property "Value" "TS-1187A-B-A-B"
-			(at 52.07 154.178 0)
+			(at 51.816 153.67 0)
 			(effects
 				(font
@@
 			)
 		)
-		(property "Datasheet" "http://www.apem.com/int/index.php?controller=attachment&id_attachment=1371"
+		(property "Datasheet" "~"
 			(at 49.53 153.67 0)
 			(effects
@@
 			)
 		)
-		(property "Description" "MEC 5E single pole normally-open tactile switch"
-			(at 49.53 161.29 0)
+		(property "Description" "Push button switch, generic, two pins"
+			(at 49.53 158.75 0)
 			(effects
 				(font
@@
 		(pin "1"
 		)
-		(pin "4"
-		)
-		(pin "3"
-		)
 		(pin "2"

Commit message: :sparkles: Update schematic
Connections:
- net D+: now also R4.2; no longer R1.2
- net D-: now also R1.2; no longer R4.2
Changed lines of the file:
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@@
 	)
 	(label "D-"
-		(at 82.55 67.31 180)
+		(at 82.55 59.69 180)
 		(fields_autoplaced yes)
 		(effects
@@
 	)
 	(label "D+"
-		(at 82.55 59.69 180)
+		(at 82.55 67.31 180)
 		(fields_autoplaced yes)
 		(effects
